Commit message: add a little script to do the visualization

File: models/urdf/harpy.urdf (robot description, URDF)
Before this commit: robot harpy, 12 links, 11 joints
Links:
- link FemurLeft: geometry visual mesh filename=../meshes/Femur.OBJ
- link FemurRight: geometry visual mesh filename=../meshes/Femur.OBJ
- link FootLeft: geometry visual mesh filename=../meshes/Foot.OBJ
- link FootRight: geometry visual mesh filename=../meshes/Foot.OBJ
- link HipLeft: geometry visual mesh filename=../meshes/Hip.OBJ
- link HipRight: geometry visual mesh filename=../meshes/Hip.OBJ
- link ThrusterLeft: geometry visual mesh filename=../meshes/Thruster.OBJ
- link ThrusterRight: geometry visual mesh filename=../meshes/Thruster.OBJ
- link TibiaLeft: geometry visual mesh filename=../meshes/Tibia.OBJ
- link TibiaRight: geometry visual mesh filename=../meshes/Tibia.OBJ
- link Torso: geometry visual mesh filename=../meshes/TorsoPelvis.OBJ

Commit message: remove spurious world frame

File: models/urdf/harpy.urdf (robot description, URDF)
Before this commit: robot harpy, 12 links, 11 joints
Links:
- removed link World
Joints:
- removed joint Torso_Base

Commit message: generate new masses and inertias assuming density of water

File: models/urdf/harpy.urdf (robot description, URDF)
Before this commit: robot harpy, 11 links, 10 joints
Links:
- link FemurLeft: mass 1.0 -> 0.2
- link FemurRight: mass 1.0 -> 0.2
- link FootLeft: mass 1.0 -> 0.09
- link FootRight: mass 1.0 -> 0.09
- link HipLeft: mass 1.0 -> 0.27
- link HipRight: mass 1.0 -> 0.27
- link ThrusterLeft: mass 1.0 -> 0.36
- link ThrusterRight: mass 1.0 -> 0.36
- link TibiaLeft: mass 1.0 -> 0.28
- link TibiaRight: mass 1.0 -> 0.28
- link Torso: mass 1.0 -> 2.3

Commit message: add (point contact) collisions

File: models/urdf/harpy.urdf (robot description, URDF)
Before this commit: robot harpy, 11 links, 10 joints
Links:
- link FemurLeft: geometry collision mesh filename=../meshes/Femur.OBJ; visual mesh filename=../meshes/Femur.OBJ
- link FemurRight: geometry collision mesh filename=../meshes/Femur.OBJ; visual mesh filename=../meshes/Femur.OBJ
- link FootLeft: geometry collision mesh filename=../meshes/Foot.OBJ; visual mesh filename=../meshes/Foot.OBJ
- link FootRight: geometry collision mesh filename=../meshes/Foot.OBJ; visual mesh filename=../meshes/Foot.OBJ
- link HipLeft: geometry collision mesh filename=../meshes/Hip.OBJ; visual mesh filename=../meshes/Hip.OBJ
- link HipRight: geometry collision mesh filename=../meshes/Hip.OBJ; visual mesh filename=../meshes/Hip.OBJ
- link ThrusterLeft: geometry collision mesh filename=../meshes/Thruster.OBJ; visual mesh filename=../meshes/Thruster.OBJ
- link ThrusterRight: geometry collision mesh filename=../meshes/Thruster.OBJ; visual mesh filename=../meshes/Thruster.OBJ
- link TibiaLeft: geometry collision mesh filename=../meshes/Tibia.OBJ; visual mesh filename=../meshes/Tibia.OBJ
- link TibiaRight: geometry collision mesh filename=../meshes/Tibia.OBJ; visual mesh filename=../meshes/Tibia.OBJ
- link Torso: geometry collision mesh filename=../meshes/TorsoPelvis.OBJ; visual mesh filename=../meshes/TorsoPelvis.OBJ
