Commit message: added yaml config file for sim settings

File: models/urdf/harpy_planar_CIMPC_staircase.urdf (robot description, URDF)
Before this commit: robot harpy, 12 links, 12 joints
Links:
- added link Staircase, mass 1000; collision mesh filename=../meshes/AmberLabStaircase.OBJ; visual mesh filename=../meshes/AmberLabStaircase.OBJ
Joints:
- added joint World_Staircase: type fixed, parent world, child Staircase, origin xyz=0.0 0.0 0.0 rpy=0.0 0.0 1.5708

Commit message: added front flipping to list of CIMPC behaviors. added option to see the reference trajectory.

File: models/urdf/harpy_planar_CIMPC_staircase.urdf (robot description, URDF)
Before this commit: robot harpy, 13 links, 13 joints
Links:
- link Staircase: geometry collision mesh filename=../meshes/AmberLabStaircase_2inFillet.OBJ; visual mesh filename=../meshes/AmberLabStaircase_2inFillet.OBJ
